File: pcb/cornia.kicad_pcb (KiCad board)
At the start: 2 copper layers, 159.3 x 108.3 mm, 65 parts, among them SW1 SW_Push, SW10 SW_Push, SW11 SW_Push, SW12 SW_Push, SW13 SW_Push, SW14 SW_Push, SW15 SW_Push, SW16 SW_Push, SW17 SW_Push, SW18 SW_Push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

Commit message: Finish PCB, add fab output, update doc
Routing:
- net GND: vias 522 -> 502
Other:
- board text added: "CORNIA"
- board text added: "designed by Vaarai"
- board text added: "github.com/Vaarai"
- board text removed: "TRRS"
