File: pcb/cornia.kicad_pcb (KiCad board)
At the start: 2 copper layers, 321.4 x 125.3 mm, 168 parts, among them J1 MJ-4PP-9, J2 OLED, J3 MJ-4PP-9, J4 OLED, SW1 SW_PUSH, SW10 SW_PUSH, SW11 SW_PUSH, SW12 SW_PUSH, SW13 SW_PUSH, SW14 SW_PUSH, SW15 SW_PUSH, SW16 SW_PUSH, SW17 SW_PUSH, SW18 SW_PUSH, SW19 SW_PUSH, SW2 SW_PUSH, SW20 SW_PUSH, SW21 SW_PUSH, SW22 SW_PUSH, SW23 SW_PUSH, SW24 SW_PUSH, SW25 SW_PUSH, SW26 SW_PUSH, SW27 SW_PUSH, SW28 SW_PUSH, SW29 SW_PUSH, SW3 SW_PUSH, SW30 SW_PUSH, SW31 SW_PUSH, SW32 SW_PUSH, SW33 SW_PUSH, SW34 SW_PUSH, SW35 SW_PUSH, SW36 SW_PUSH, SW37 SW_PUSH, SW38 SW_PUSH, SW39 SW_PUSH, SW4 SW_PUSH, SW40 SW_PUSH, SW41 SW_PUSH, SW42 SW_PUSH, SW5 SW_PUSH, SW6 SW_PUSH, SW7 SW_PUSH, SW8 SW_PUSH, SW9 SW_PUSH, U1 ProMicro, U2 ProMicro

Commit message: [PCB] Remove mounting Hole and give space in front of USB connector
Parts:
- removed the Ref** at (175.6, 67.8)
- removed the Ref** at (62.6, 81.8)
- removed the Ref** at (88.6, 129.8)
- removed the Ref** at (169.6, 127.8)
- removed the Ref** at (239.1, 127.8)
- removed the Ref** at (320.1, 130.3)
- removed the Ref** at (346.1, 81.8)
- removed the Ref** at (233.1, 67.8)
- U1, U2: value ProMicro -> ProMicro_r
Routing:
- net GNDA: vias 379 -> 362
- net GND: vias 399 -> 404
Other:
- outline, holes or cut-outs redrawn

Commit message: [PCB/Footprint] Increase Oled pads size + Cut PCB angle near USB
Parts:
- U1, U2: value ProMicro_r -> ProMicro
Routing:
- net VCC: track 661.6 -> 660.3 mm
- net GNDA: vias 362 -> 374
- net GND: vias 404 -> 411
Other:
- outline, holes or cut-outs redrawn
